File: SmoothieBrainz - next round.sch (EAGLE design)
At the start: 238 parts, among them IC1 LPC1769, IC7 74LVC1G04, Q1 BSL207SP, Q2 12MHz, SW1 SW_TACT_4P_B, SW3 SW_TACT_4P_B, T1 BC817, U3 USD-SOCKETUSD, X1 MSTBA2, X14 USBPTH, X2 GMSTBA2, X3 GMSTBA4, X4 1751248, X5 1751248, X6 1751248, X7 1751248

Commit message: About to fix ethernet
Parts:
- C1, C11, C12, C51, C6, C65: value .1uF -> 104
- D2: value (none) -> SS34
- IC2: value (none) -> LM2596-5
- LED1, LED2, LED3, LED4, LED9: value (none) -> GREEN
- LED10, LED11, LED8: value LED -> RED
- LED12: value VMOT -> RED
- LED5: value (none) -> GREEN; device led:LEDCHIP-LED0603 -> led:LEDSML0603
- LED6, LED7: value (none) -> RED
- R10, R11, R12, R13, R77: value (none) -> 1k
- R57: value 1.5k -> 1.5K
- U1: value (none) -> 1117-3.3
Changed lines of the file:
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@@
 <part name="C9" library="rcl" deviceset="C-EU" device="C0603" value="104"/>
 <part name="C10" library="rcl" deviceset="C-EU" device="C0603" value="104"/>
-<part name="C11" library="rcl" deviceset="C-EU" device="C0603" value=".1uF"/>
-<part name="C12" library="rcl" deviceset="C-EU" device="C0603" value=".1uF"/>
+<part name="C11" library="rcl" deviceset="C-EU" device="C0603" value="104"/>
+<part name="C12" library="rcl" deviceset="C-EU" device="C0603" value="104"/>
 <part name="C13" library="rcl" deviceset="C-EU" device="C0603" value="104"/>
 <part name="P+2" library="SparkFun" deviceset="3.3V" device=""/>
@@
 <part name="C7" library="resistor" deviceset="C-EU" device="C0603" value="10uF"/>
 <part name="L1" library="SparkFun" deviceset="INDUCTOR" device="0603" value="39nH"/>
-<part name="C6" library="rcl" deviceset="C-EU" device="C0603" value=".1uF"/>
+<part name="C6" library="rcl" deviceset="C-EU" device="C0603" value="104"/>
 <part name="R14" library="resistor" deviceset="R-US_" device="R0603" value="10K"/>
 <part name="P+19" library="SparkFun" deviceset="3.3V" device=""/>
@@
 <part name="SUPPLY28" library="supply2" deviceset="GND" device=""/>
 <part name="SUPPLY30" library="supply2" deviceset="GND" device=""/>
-<part name="C1" library="resistor" deviceset="C-EU" device="C0603" value=".1uF"/>
+<part name="C1" library="resistor" deviceset="C-EU" device="C0603" value="104"/>
 <part name="P+21" library="SparkFun" deviceset="3.3V" device=""/>
 <part name="VUSB" library="SparkFun" deviceset="5V" device="" value="VUSB"/>
@@
 <part name="P+30" library="SparkFun" deviceset="3.3V" device=""/>
 <part name="S1" library="SparkFun" deviceset="TAC_SWITCH" device="SMD"/>
-<part name="LED1" library="led" deviceset="LED" device="SML0603"/>
-<part name="LED2" library="led" deviceset="LED" device="SML0603"/>
-<part name="LED3" library="led" deviceset="LED" device="SML0603"/>
-<part name="LED4" library="led" deviceset="LED" device="SML0603"/>
-<part name="R10" library="resistor" deviceset="R-US_" device="R0603"/>
-<part name="R11" library="resistor" deviceset="R-US_" device="R0603"/>
-<part name="R12" library="resistor" deviceset="R-US_" device="R0603"/>
-<part name="R13" library="resistor" deviceset="R-US_" device="R0603"/>
+<part name="LED1" library="led" deviceset="LED" device="SML0603" value="GREEN"/>
+<part name="LED2" library="led" deviceset="LED" device="SML0603" value="GREEN"/>
+<part name="LED3" library="led" deviceset="LED" device="SML0603" value="GREEN"/>
+<part name="LED4" library="led" deviceset="LED" device="SML0603" value="GREEN"/>
+<part name="R10" library="resistor" deviceset="R-US_" device="R0603" value="1k"/>
+<part name="R11" library="resistor" deviceset="R-US_" device="R0603" value="1k"/>
+<part name="R12" library="resistor" deviceset="R-US_" device="R0603" value="1k"/>
+<part name="R13" library="resistor" deviceset="R-US_" device="R0603" value="1k"/>
 <part name="SUPPLY65" library="supply2" deviceset="GND" device=""/>
 <part name="R3" library="resistor" deviceset="R-US_" device="R0603" value="10K"/>
@@
 <part name="VUSB2" library="SparkFun" deviceset="5V" device="" value="VUSB"/>
 <part name="P+27" library="SparkFun" deviceset="3.3V" device=""/>
-<part name="C65" library="resistor" deviceset="C-EU" device="C0603" value=".1uF"/>
+<part name="C65" library="resistor" deviceset="C-EU" device="C0603" value="104"/>
 <part name="C64" library="resistor" deviceset="C-EU" device="C0603" value="10uF"/>
 <part name="SUPPLY59" library="supply2" deviceset="GND" device=""/>
-<part name="LED9" library="led" deviceset="LED" device="SML0603"/>
-<part name="R77" library="resistor" deviceset="R-US_" device="R0603"/>
+<part name="LED9" library="led" deviceset="LED" device="SML0603" value="GREEN"/>
+<part name="R77" library="resistor" deviceset="R-US_" device="R0603" value="1k"/>
 <part name="D1" library="microbuilder" deviceset="DIODE" device="SMA" value="MBRA210LT3"/>
 <part name="U$3" library="SparkFun" deviceset="5V" device=""/>
-<part name="IC2" library="linear" deviceset="LM2596S" device=""/>
+<part name="IC2" library="linear" deviceset="LM2596S" device="" value="LM2596-5"/>
 <part name="L2" library="SparkFun-Passives" deviceset="INDUCTOR" device="PWR" value="33uH"/>
-<part name="D2" library="dp_devices" deviceset="DIODE" device="-DO-214AC"/>
+<part name="D2" library="dp_devices" deviceset="DIODE" device="-DO-214AC" value="SS34"/>
 <part name="C26" library="rcl" deviceset="CPOL-EU" device="E2.5-7" value="220u"/>
 <part name="C27" library="rcl" deviceset="CPOL-EU" device="E2.5-7" value="220u"/>
@@
 <part name="SUPPLY4" library="supply2" deviceset="GND" device=""/>
 <part name="JP5" library="SparkFun-Connectors" deviceset="M05" device="NO_SILK"/>
-<part name="LED5" library="led" deviceset="LED" device="CHIP-LED0603"/>
+<part name="LED5" library="led" deviceset="LED" device="SML0603" value="GREEN"/>
 <part name="R18" library="resistor" deviceset="R-US_" device="R0603" value="1k"/>
 <part name="U3" library="SparkFun-Connectors_PETERMICROSDEBAY" deviceset="USD-SOCKET" device="USD"/>
@@
 <part name="R30" library="resistor" deviceset="R-EU_" device="R0603" value="100k"/>
 <part name="R32" library="resistor" deviceset="R-EU_" device="R0603" value="1.5k"/>
-<part name="LED6" library="led" deviceset="LED" device="SML0603"/>
+<part name="LED6" library="led" deviceset="LED" device="SML0603" value="RED"/>
 <part name="X2" library="con-phoenix-762" deviceset="GMSTBA2" device=""/>
 <part name="X3" library="con-phoenix-762" deviceset="GMSTBA4" device=""/>
@@
 <part name="R36" library="resistor" deviceset="R-EU_" device="R0603" value="100k"/>
 <part name="GND15" library="supply1" deviceset="GND" device=""/>
-<part name="LED7" library="led" deviceset="LED" device="SML0603"/>
+<part name="LED7" library="led" deviceset="LED" device="SML0603" value="RED"/>
 <part name="R37" library="resistor" deviceset="R-EU_" device="R0603" value="1.5k"/>
 <part name="X4" library="con-phoenix-350-ray" deviceset="1751248" device=""/>
@@
 <part name="P+8" library="SparkFun" deviceset="3.3V" device=""/>
 <part name="JP12" library="SparkFun-Connectors" deviceset="M04" device="LOCK"/>
-<part name="U1" library="SparkFun-PowerIC" deviceset="V_REG_LM1117" device="SOT223"/>
+<part name="U1" library="SparkFun-PowerIC" deviceset="V_REG_LM1117" device="SOT223" value="1117-3.3"/>
 <part name="SUPPLY5" library="supply2" deviceset="GND" device=""/>
 <part name="RN2" library="resistor-dil" deviceset="4R-N" device="0603-ARV" value="4k7"/>
@@
 <part name="R41" library="resistor" deviceset="R-EU_" device="R0603" value="100k"/>
 <part name="GND1" library="supply1" deviceset="GND" device=""/>
-<part name="LED8" library="led" deviceset="LED" device="SML0603" value="LED"/>
+<part name="LED8" library="led" deviceset="LED" device="SML0603" value="RED"/>
 <part name="R42" library="resistor" deviceset="R-EU_" device="R0603" value="1.5k"/>
 <part name="U$15" library="Cohesion_parts" deviceset="N-POWER-MOSFET" device="DPAK-MOSFET" value="IRLR024"/>
@@
 <part name="R44" library="resistor" deviceset="R-EU_" device="R0603" value="100k"/>
 <part name="GND2" library="supply1" deviceset="GND" device=""/>
-<part name="LED10" library="led" deviceset="LED" device="SML0603" value="LED"/>
+<part name="LED10" library="led" deviceset="LED" device="SML0603" value="RED"/>
 <part name="R45" library="resistor" deviceset="R-EU_" device="R0603" value="1.5k"/>
 <part name="U$16" library="Cohesion_parts" deviceset="N-POWER-MOSFET" device="DPAK-MOSFET" value="IRLR024"/>
@@
 <part name="R47" library="resistor" deviceset="R-EU_" device="R0603" value="100k"/>
 <part name="GND3" library="supply1" deviceset="GND" device=""/>
-<part name="LED11" library="led" deviceset="LED" device="SML0603" value="LED"/>
+<part name="LED11" library="led" deviceset="LED" device="SML0603" value="RED"/>
 <part name="R48" library="resistor" deviceset="R-EU_" device="R0603" value="1.5k"/>
 <part name="U$8" library="RepRapjr" deviceset="POLOLU_A4983CARRIER" device=""/>
@@
 <part name="R53" library="resistor" deviceset="R-US_" device="R0603" value="22R"/>
 <part name="SUPPLY56" library="supply2" deviceset="GND" device=""/>
-<part name="C51" library="resistor" deviceset="C-EU" device="C0603" value=".1uF"/>
+<part name="C51" library="resistor" deviceset="C-EU" device="C0603" value="104"/>
 <part name="SUPPLY57" library="supply2" deviceset="GND" device=""/>
 <part name="P+18" library="SparkFun" deviceset="3.3V" device=""/>
@@
 <part name="C23" library="resistor" deviceset="CPOL-EU" device="153CLV-0605" value="100u"/>
 <part name="C24" library="resistor" deviceset="CPOL-EU" device="153CLV-0605" value="100u"/>
-<part name="LED12" library="led" deviceset="LED" device="SML0603" value="VMOT"/>
-<part name="R57" library="resistor" deviceset="R-EU_" device="R0603" value="1.5k"/>
+<part name="LED12" library="led" deviceset="LED" device="SML0603" value="RED"/>
+<part name="R57" library="resistor" deviceset="R-EU_" device="R0603" value="1.5K"/>
 <part name="JP16" library="SparkFun-Connectors" deviceset="M02" device="LOCK"/>
 <part name="JP21" library="SparkFun-Connectors" deviceset="M02" device="LOCK"/>
