File: C3D ReMix rev2.brd (EAGLE design)
At the start: 101 x 101 mm, 238 parts, among them IC1 LPC1769, IC2 LM2596-5, IC7 74LVC1G04, Q1 BSL207SP, Q2 12MHz, SW1 SW_TACT_4P_B, SW3 SW_TACT_4P_B, T1 BC817, U1 1117-3.3, U3 USD-SOCKETUSD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

Commit message: Almost done, but need to replace 220uF caps with SMD
Parts:
- removed U$18, U$19, U$20: FIDUCIAL, adafruit:FIDUCIAL_1MM
- removed X2: GMSTBA2, con-phoenix-762:GMSTBA2
- removed X3: GMSTBA4, con-phoenix-762:GMSTBA4
- removed X4, X5, X6, X7: 1751248, con-phoenix-350-ray:1751248
- added C15, C16: (no value), resistor:153CLV-0810
- added X8: 1751303, con-phoenix-350-ray:1751303
- added X9: GMSTBA6, con-phoenix-762:GMSTBA6
- C23, C24: value 100u -> 100uF
- R16, R28, R29, R31, R4: device adafruit:R0603 -> resistor:R0603
- R20, R34, R39, R50, R52: value 10k -> 10K
- R21, R22, R23, R24, R5, R6: value 10k -> 10K; device adafruit:R0603 -> resistor:R0603
- R57, R7: value 1.5K -> 1.5k
- moved D13 1.91 mm to (30.2, 8.00)
- moved JP23 1.91 mm to (32.4, 8.51)
- moved LED11 1.91 mm to (32.9, 23.5)
- moved R46 1.91 mm to (35.1, 23.8)
- moved R47 1.91 mm to (30.6, 23.8)
- moved R48 1.91 mm to (33.2, 20.8)
- moved U$16 1.91 mm to (32.9, 15.2)
- moved JP22 1.27 mm to (25.4, 8.51)
- moved D6 1.27 mm to (23.2, 8.00)
- moved LED10 1.27 mm to (25.9, 23.5)
- moved R43 1.27 mm to (28.1, 23.8)
- moved R44 1.27 mm to (23.7, 23.8)
- moved R45 1.27 mm to (26.2, 20.8)
- moved U$15 1.27 mm to (25.9, 15.2)
- moved JP21 0.64 mm to (18.4, 8.51)
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Connections:
- net 24V: now also X9.1; no longer X2.1
- net E1-CONTROL: now also X8.2; no longer X4.2
- net E2-CONTROL: now also X8.4; no longer X5.2
- net E3-CONTROL: now also X8.6; no longer X6.2
- net E4-CONTROL: now also X8.8; no longer X7.2
- net GND: now also X9.2, X9.4; no longer X2.2, X3.2
- net HEATBED-CONTROL: now also X9.6; no longer X3.4
- net HEATBEDVIN: now also X9.3, X9.5; no longer X3.1, X3.3
- net HEATERVIN: now also X8.1, X8.3, X8.5, X8.7; no longer X4.1, X5.1, X6.1, X7.1
Routing:
- net GND: track 814.6 -> 778.2 mm, vias 204 -> 205
- net ENET_TX_EN: track 43.0 -> 28.6 mm, vias 0 -> 2
- net 3.3V: track 679.9 -> 694.3 mm, vias 31 -> 32
- net ENET_TXD1: track 44.6 -> 30.5 mm, vias 1 -> 0
- net ENET_CRS: track 45.8 -> 32.1 mm
- net N$77: track 9.91 -> 23.6 mm, vias 0 -> 1
- net ENET_TXD0: track 49.7 -> 36.7 mm
- net ENET_RXD0: track 36.3 -> 27.1 mm, vias 0 -> 1
- net ENET_RXD1: track 37.1 -> 28.4 mm, vias 0 -> 1
- net E1-CONTROL: track 17.3 -> 10.0 mm
- net 24V: track 314.4 -> 308.5 mm
- net ENET_MDC: track 22.4 -> 28.2 mm
- net ENET_MDIO: track 16.9 -> 22.6 mm, vias 1 -> 2
- net PLAY_LED: track 81.3 -> 77.1 mm
- net HEATBEDVIN: track 33.3 -> 29.7 mm
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Other:
- board text added: "Manufactured by Cohesion3D"
- board text added: "With Special thanks to: Ross Bagley, Samer Najia, Brian Bland, and Mark Harris"
- board text removed: "BSL207SP"

Commit message: 1/2 Cap 220uF Converted
Parts:
- removed C26: 220u, rcl:E2,5-7
- moved C27 38.1 mm to (-9.66, 55.0)
- moved C16 3.05 mm to (27.9, 55.8)
- moved IC2 1.27 mm to (30.8, 65.3)
- turned C15 to 180 degrees
Connections:
- net 24V: now also C15.+; no longer C26.+
- net GND: now also C15.-; no longer C26.-
Routing:
- net 5VREG: track 27.8 -> 15.5 mm
- net GND: track 778.2 -> 774.7 mm
- net N$9: track 8.78 -> 5.46 mm
- net 24V: track 308.5 -> 306.4 mm

Commit message: Rev2, Huge Amount of stuff added
Parts:
- removed C27: 220u, rcl:E2,5-7
- added R56: 10k, resistor:R0603
- C15, C16: value (none) -> 220uF
- U$13, U$14, U$15, U$16: value IRLR024 -> SUD50N04
- moved U$17 2.82 mm to (1.65, 24.0)
- moved D3 1.53 mm to (37.4, 57.4)
- moved C24 0.90 mm to (36.2, 50.2)
- moved C16 0.52 mm to (28.4, 55.5)
- moved JP17 0.51 mm to (59.1, 14.0)
- moved L2 0.36 mm to (17.2, 58.0)
- moved X9 0.25 mm to (1.91, 50.0)
- moved U1 0.25 mm to (24.9, 47.8)
- moved D15 0.13 mm to (6.35, 26.1)
Connections:
- net USB_D+ renamed USB_P
- net USB_D- renamed USB_N
- net 5V: now also R56.2
- net 5VREG: now also C16.+; no longer C27.+
- net GND: now also C16.-; no longer C27.-
- net N$56: now also R56.1
Routing:
- net 5V: track 284.3 -> 305.3 mm
- net GND: track 774.7 -> 760.4 mm
- net N$56: track 10.8 -> 18.1 mm
- net 5VREG: track 15.5 -> 20.1 mm
- net N$34: track 2.00 -> 3.74 mm
- net N$17: track 2.00 -> 3.68 mm
- net N$53: track 2.00 -> 3.68 mm
- net N$33: track 2.00 -> 3.68 mm
- net N$15: track 2.00 -> 3.68 mm
- net N$54: track 2.00 -> 3.62 mm
- net N$36: track 2.00 -> 3.62 mm
- net N$50: track 2.00 -> 3.55 mm
- net N$46: track 2.00 -> 3.55 mm
- net N$45: track 2.00 -> 3.55 mm
- net N$8: track 2.00 -> 3.56 mm
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Other:
- outline, holes or cut-outs redrawn
- board text added: "+24V MAX"
- board text added: "MOSFETS"
- board text added: "With special thanks to: Ross Bagley, Samer Najia, Brian Bland, and Mark Harris"
- board text removed: "(24V MAX)"
- board text removed: "MBRA210LT3"
- board text removed: "With Special thanks to: Ross Bagley, Samer Najia, Brian Bland, and Mark Harris"
